Commit message: added all joints to urdf

File: ra1_pro/urdf/ra1_pro.urdf (robot description, URDF)
Before this commit: robot alfred, 6 links, 5 joints
Links:
- added link camera; visual box size=0.025 .04 .035
- added link gripper_left; visual box size=0.01 .02 .05
- added link gripper_right; visual box size=0.01 .02 .05
- added link wrist_box_s2; visual box size=0.04 .05 .035
- added link wrist_s2; visual box size=0.017 .05 .075
Joints:
- added joint _wrist_box_s2_to_camera: type fixed, parent wrist_box_s2, child camera, origin xyz=0.04 0 0.04 rpy=0 -0.34906585039887 0
- added joint wrist_s2_to_gripper_left: type prismatic, parent wrist_s2, child gripper_left, origin xyz=0 -0.025 .075, axis 0 1 0, limit lower=0 upper=0.015 effort=1000.0 velocity=0.5
- added joint wrist_s2_to_gripper_right: type prismatic, parent wrist_s2, child gripper_right, origin xyz=0 0.025 .075, axis 0 1 0, limit lower=-0.015 upper=0 effort=1000.0 velocity=0.5
- added joint wrist_s2_to_wrist_box_s2: type fixed, parent wrist_s2, child wrist_box_s2, origin xyz=0.0085 0 0
- added joint wrist_s3_to_wrist_s2: type continuous, parent wrist_s3, child wrist_s2, origin xyz=0 0 0.065, axis 0 0 1
- joint cylinder_to_base_s6: limit (none) -> lower=0.0 upper=0.548 effort=1000.0 velocity=0.5; type continuous -> revolute

Commit message: finished urdf with all joint limits

File: ra1_pro/urdf/ra1_pro.urdf (robot description, URDF)
Before this commit: robot alfred, 11 links, 10 joints
Links:
- removed link base_link
- added link base; visual box size=0.27 .25 .065
Joints:
- removed joint base_s6_to_shoulder_s5
- removed joint cylinder_to_base_s6
- removed joint elbow_s4_to_wrist_s3
- removed joint shoulder_s5_to_elbow_s4
- removed joint wrist_s2_to_gripper_left
- removed joint wrist_s2_to_gripper_right
- removed joint wrist_s3_to_wrist_s2
- added joint gripper_finger_left: type prismatic, parent wrist_s2, child gripper_left, origin xyz=0 -0.025 .075, axis 0 1 0, limit lower=0 upper=0.015 effort=1000.0 velocity=0.5
- added joint gripper_finger_right: type prismatic, parent wrist_s2, child gripper_right, origin xyz=0 0.025 .075, axis 0 1 0, limit lower=-0.015 upper=0 effort=1000.0 velocity=0.5
- added joint servo_2: type revolute, parent wrist_s3, child wrist_s2, origin xyz=0 0 0.065 rpy=0 0 -3.1415926535898, axis 0 0 1, limit lower=-3.1415926535898 upper=0.0 effort=1000.0 velocity=0.5
- added joint servo_3: type revolute, parent elbow_s4, child wrist_s3, origin xyz=0 0 0.08, axis 0 1 0, limit lower=-1.7453292519943 upper=1.7453292519943 effort=1.0 velocity=0.5
- added joint servo_4: type revolute, parent shoulder_s5, child elbow_s4, origin xyz=0 0 0.08, axis 0 1 0, limit lower=-1.7453292519943 upper=1.7453292519943 effort=1000.0 velocity=0.5
- added joint servo_5: type revolute, parent base_s6, child shoulder_s5, origin xyz=0 0 0.015, axis 0 1 0, limit lower=-1.7453292519943 upper=1.7453292519943 effort=1000.0 velocity=0.5
- added joint servo_6: type revolute, parent cylinder, child base_s6, origin xyz=0 0 0.055, axis 0 0 1, limit lower=-1.7453292519943 upper=1.7453292519943 effort=1000.0 velocity=0.5
- joint box_to_cylinder: parent base_link -> base

Commit message: created moveit config

File: ra1_pro/urdf/ra1_pro.urdf (robot description, URDF)
Before this commit: robot alfred, 11 links, 10 joints
Links:
- link base: geometry collision box size=0.27 .25 .065; visual box size=0.27 .25 .065
- link base_s6: geometry collision box size=0.06 .04 .035; visual box size=0.06 .04 .035
- link camera: geometry collision box size=0.025 .04 .035; visual box size=0.025 .04 .035
- link cylinder: geometry collision cylinder length=0.035 radius=0.085; visual cylinder length=0.035 radius=0.085
- link elbow_s4: geometry collision box size=0.03 .04 .12; visual box size=0.03 .04 .12
- link gripper_left: geometry collision box size=0.01 .02 .05; visual box size=0.01 .02 .05
- link gripper_right: geometry collision box size=0.01 .02 .05; visual box size=0.01 .02 .05
- link shoulder_s5: geometry collision box size=0.025 .06 .105; visual box size=0.025 .06 .105
- link wrist_box_s2: geometry collision box size=0.04 .05 .035; visual box size=0.04 .05 .035
- link wrist_s2: geometry collision box size=0.017 .05 .075; visual box size=0.017 .05 .075
- link wrist_s3: geometry collision box size=0.025 .06 .07; visual box size=0.025 .06 .07

Commit message: changes

File: ra1_pro/urdf/ra1_pro.urdf (robot description, URDF)
Before this commit: robot alfred, 11 links, 10 joints
Joints:
- joint gripper_finger_left: limit lower=0 upper=0.015 effort=1000.0 velocity=0.5 -> lower=0 upper=0.015 effort=1000.0 velocity=0.9
- joint gripper_finger_right: limit lower=-0.015 upper=0 effort=1000.0 velocity=0.5 -> lower=-0.015 upper=0 effort=1000.0 velocity=0.9
- joint servo_2: limit lower=-3.1415926535898 upper=0.0 effort=1000.0 velocity=0.5 -> lower=-3.1415926535898 upper=0.0 effort=1000.0 velocity=0.9
- joint servo_3: limit lower=-1.7453292519943 upper=1.7453292519943 effort=1.0 velocity=0.5 -> lower=-1.7453292519943 upper=1.7453292519943 effort=1.0 velocity=0.9
- joint servo_4: axis 0 1 0 -> 0 -1 0; limit lower=-1.7453292519943 upper=1.7453292519943 effort=1000.0 velocity=0.5 -> lower=-1.7453292519943 upper=1.7453292519943 effort=1000.0 velocity=0.9
- joint servo_5: limit lower=-1.7453292519943 upper=1.7453292519943 effort=1000.0 velocity=0.5 -> lower=-1.7453292519943 upper=1.7453292519943 effort=1000.0 velocity=0.9
- joint servo_6: limit lower=-1.7453292519943 upper=1.7453292519943 effort=1000.0 velocity=0.5 -> lower=-1.7453292519943 upper=1.7453292519943 effort=1000.0 velocity=0.9

Commit message: fixed moveit and controller

File: ra1_pro/urdf/ra1_pro.urdf (robot description, URDF)
Before this commit: robot alfred, 11 links, 10 joints
Joints:
- joint servo_2: limit lower=-3.1415926535898 upper=0.0 effort=1000.0 velocity=0.9 -> lower=-1.7453292519943 upper=1.7453292519943 effort=1000.0 velocity=0.9; origin xyz=0 0 0.065 rpy=0 0 -3.1415926535898 -> xyz=0 0 0.065 rpy=0 0 1.5707963267949

Commit message: working on smach

File: ra1_pro/urdf/ra1_pro.urdf (robot description, URDF)
Before this commit: robot alfred, 11 links, 10 joints
Joints:
- joint gripper_finger_right: mimic (none) -> joint=gripper_finger_left multiplier=-1.0

Commit message: refinement

File: ra1_pro/urdf/ra1_pro.urdf (robot description, URDF)
Before this commit: robot alfred, 11 links, 10 joints
Joints:
- joint servo_2: limit lower=-1.7453292519943 upper=1.7453292519943 effort=1000.0 velocity=0.9 -> lower=-1.5707963267949 upper=1.5707963267949 effort=1000.0 velocity=0.9
- joint servo_3: limit lower=-1.7453292519943 upper=1.7453292519943 effort=1.0 velocity=0.9 -> lower=-1.5707963267949 upper=1.5707963267949 effort=1.0 velocity=0.9
- joint servo_4: limit lower=-1.7453292519943 upper=1.7453292519943 effort=1000.0 velocity=0.9 -> lower=-1.5707963267949 upper=1.5707963267949 effort=1000.0 velocity=0.9
- joint servo_5: limit lower=-1.7453292519943 upper=1.7453292519943 effort=1000.0 velocity=0.9 -> lower=-1.5707963267949 upper=1.5707963267949 effort=1000.0 velocity=0.9
- joint servo_6: limit lower=-1.7453292519943 upper=1.7453292519943 effort=1000.0 velocity=0.9 -> lower=-1.5707963267949 upper=1.5707963267949 effort=1000.0 velocity=0.9
